File: achterart/achterart.kicad_pcb (KiCad board)
At the start: 2 copper layers, 139.7 x 100.3 mm, 63 parts, among them J1 S4B-PH-SM4-TB(LF)(SN), J10 PH1-04-UA, J11 PH1-04-UA, J12 PH1-04-UA, J13 PH1-04-UA, J14 PH1-04-UA, J15 PH1-04-UA, J16 PH1-04-UA, J17 UJ2-BH-1-TH, J18 PH2-06-UA, J2 S4B-PH-SM4-TB(LF)(SN), J3 S4B-PH-SM4-TB(LF)(SN), J4 S4B-PH-SM4-TB(LF)(SN), J5 S4B-PH-SM4-TB(LF)(SN), J6 S4B-PH-SM4-TB(LF)(SN), J7 S4B-PH-SM4-TB(LF)(SN), J8 S4B-PH-SM4-TB(LF)(SN), J9 PH1-04-UA, U1 TLV74033PDBVR, U2 TLV75801PDBVT, U3 ESD224DQA, U4 ESD224DQA, U5 ESD224DQA, U6 ESD224DQA, U7 CH348L, Y1 8MHz

Commit message: Add JST 3d model
Pretty sure I can't distribute it, so it's just gonna be useless
to everyone not on my computer.
Parts:
- J1, J2, J3, J4, J5, J6, J7, J8: footprint Connector_JST:JST_PH_S4B-PH-SM4-TB_1x04-1MP_P2.00mm_Horizontal -> dumb-jst-shit:JST_PH_S4B-PH-SM4-TB_1x04-1MP_P2.00mm_Horizontal_Model
